File: schematics/Components.sch (KiCad schematic (older format))
At the start: 10 parts, among them Q1 RFD3055LE, Q2 RFD3055LE, Q3 RFD3055LE, U2 LD1117_3V3

Commit message: Change Resistor footprint
Parts:
- R1, R2, R3: footprint Resistor_THT:R_Axial_DIN0207_L6.3mm_D2.5mm_P5.08mm_Vertical -> Resistor_THT:R_Axial_DIN0207_L6.3mm_D2.5mm_P7.62mm_Horizontal
Changed lines of the file:
@@
 $Descr User 8268 5827
 encoding utf-8
-Sheet 2 2
+Sheet 1 1
 Title "Generic RGB LED strip controller"
 Date ""
@@
 F 0 "R1" H 4009 2246 50  0000 L CNN
 F 1 "10k" H 4009 2155 50  0000 L CNN
-F 2 "Resistor_THT:R_Axial_DIN0207_L6.3mm_D2.5mm_P5.08mm_Vertical" H 3950 2200 50  0001 C CNN
+F 2 "Resistor_THT:R_Axial_DIN0207_L6.3mm_D2.5mm_P7.62mm_Horizontal" H 3950 2200 50  0001 C CNN
 F 3 "~" H 3950 2200 50  0001 C CNN
 	1    3950 2200
@@
 F 0 "R2" H 4009 2796 50  0000 L CNN
 F 1 "10k" H 4009 2705 50  0000 L CNN
-F 2 "Resistor_THT:R_Axial_DIN0207_L6.3mm_D2.5mm_P5.08mm_Vertical" H 3950 2750 50  0001 C CNN
+F 2 "Resistor_THT:R_Axial_DIN0207_L6.3mm_D2.5mm_P7.62mm_Horizontal" H 3950 2750 50  0001 C CNN
 F 3 "~" H 3950 2750 50  0001 C CNN
 	1    3950 2750
@@
 F 0 "R3" H 4009 3346 50  0000 L CNN
 F 1 "10k" H 4009 3255 50  0000 L CNN
-F 2 "Resistor_THT:R_Axial_DIN0207_L6.3mm_D2.5mm_P5.08mm_Vertical" H 3950 3300 50  0001 C CNN
+F 2 "Resistor_THT:R_Axial_DIN0207_L6.3mm_D2.5mm_P7.62mm_Horizontal" H 3950 3300 50  0001 C CNN
 F 3 "~" H 3950 3300 50  0001 C CNN
 	1    3950 3300
