File: schematics/D1mini/D1mini.sch (KiCad schematic (older format))
At the start: 2 parts

Commit message: Change MOSFET, annotate schematics
Parts:
- gave numbers to parts that had none: 2
Changed lines of the file:
@@
 $EndSheet
 $Comp
-L MCU_Module:WeMos_D1_mini U?
+L MCU_Module:WeMos_D1_mini U1
 U 1 1 60EFBAE9
 P 3600 2550
-F 0 "U?" H 3800 1950 50  0000 C CNN
+F 0 "U1" H 3800 1950 50  0000 C CNN
 F 1 "WeMos_D1_mini" V 3400 1900 50  0000 L CNN
 F 2 "Module:WEMOS_D1_mini_light" H 3600 1400 50  0001 C CNN
@@
 	2850 2850 2850 3400
 $Comp
-L power:GND #PWR?
+L power:GND #PWR0101
 U 1 1 60F14A50
 P 1650 2650
-F 0 "#PWR?" H 1650 2400 50  0001 C CNN
+F 0 "#PWR0101" H 1650 2400 50  0001 C CNN
 F 1 "GND" V 1655 2522 50  0000 R CNN
 F 2 "" H 1650 2650 50  0001 C CNN
@@
 $EndComp
 $Comp
-L Connector:Barrel_Jack J?
+L Connector:Barrel_Jack J1
 U 1 1 60F12523
 P 1350 2550
-F 0 "J?" H 1250 2550 50  0000 C CNN
+F 0 "J1" H 1250 2550 50  0000 C CNN
 F 1 "Barrel_Jack" H 1350 2350 50  0000 C CNN
 F 2 "" H 1400 2510 50  0001 C CNN
@@
 	1650 2450 2100 2450
 $Comp
-L power:+12V #PWR?
+L power:+12V #PWR0102
 U 1 1 60F0705D
 P 2100 2700
-F 0 "#PWR?" H 2100 2550 50  0001 C CNN
+F 0 "#PWR0102" H 2100 2550 50  0001 C CNN
 F 1 "+12V" H 2115 2873 50  0000 C CNN
 F 2 "" H 2100 2700 50  0001 C CNN
@@
 	2100 2450 2250 2450
 $Comp
-L power:GND #PWR?
+L power:GND #PWR0103
 U 1 1 60F02616
 P 2800 2450
-F 0 "#PWR?" H 2800 2200 50  0001 C CNN
+F 0 "#PWR0103" H 2800 2200 50  0001 C CNN
 F 1 "GND" V 2805 2322 50  0000 R CNN
 F 2 "" H 2800 2450 50  0001 C CNN
@@
 $EndComp
 $Comp
-L power:GND #PWR?
+L power:GND #PWR0104
 U 1 1 60F03102
 P 3600 1750
-F 0 "#PWR?" H 3600 1500 50  0001 C CNN
+F 0 "#PWR0104" H 3600 1500 50  0001 C CNN
 F 1 "GND" H 3605 1577 50  0000 C CNN
 F 2 "" H 3600 1750 50  0001 C CNN

Commit message: Assign footprints
Parts:
- J1: footprint (none) -> Connector_BarrelJack:BarrelJack_Horizontal
Changed lines of the file:
@@
 F 0 "J1" H 1250 2550 50  0000 C CNN
 F 1 "Barrel_Jack" H 1350 2350 50  0000 C CNN
-F 2 "" H 1400 2510 50  0001 C CNN
+F 2 "Connector_BarrelJack:BarrelJack_Horizontal" H 1400 2510 50  0001 C CNN
 F 3 "~" H 1400 2510 50  0001 C CNN
 	1    1350 2550
