File: schematics/ESP12/ESP12.sch (KiCad schematic (older format))
At the start: 2 parts, among them J1 Barrel_Jack

Commit message: Annotate ESP12, connect ground
Parts:
- gave numbers to parts that had none: 1
Connections:
- net GND: now also U1.15 (GND)
Changed lines of the file:
@@
 L power:GND #PWR0104
 U 1 1 60F03102
-P 4900 1750
-F 0 "#PWR0104" H 4900 1500 50  0001 C CNN
-F 1 "GND" H 4905 1577 50  0000 C CNN
-F 2 "" H 4900 1750 50  0001 C CNN
-F 3 "" H 4900 1750 50  0001 C CNN
-	1    4900 1750
+P 5100 1850
+F 0 "#PWR0104" H 5100 1600 50  0001 C CNN
+F 1 "GND" H 5105 1677 50  0000 C CNN
+F 2 "" H 5100 1850 50  0001 C CNN
+F 3 "" H 5100 1850 50  0001 C CNN
+	1    5100 1850
 	-1   0    0    1
 $EndComp
 $Comp
-L RF_Module:ESP-12F U?
+L RF_Module:ESP-12F U1
 U 1 1 60F9FE62
 P 5100 2550
-F 0 "U?" H 5100 1669 50  0000 C CNN
-F 1 "ESP-12F" H 5100 1760 50  0000 C CNN
+F 0 "U1" H 4600 3300 50  0000 L CNN
+F 1 "ESP-12F" H 4600 3400 50  0000 L CNN
 F 2 "RF_Module:ESP-12E" H 5100 2550 50  0001 C CNN
 F 3 "http://wiki.ai-thinker.com/_media/esp8266/esp8266_series_modules_user_manual_v1.1.pdf" H 4750 2650 50  0001 C CNN
